File: PCB_DiscoF746-NG/carte_kicad_F46NG/carte_kicad_F46NG.kicad_pcb (KiCad board)
At the start: 2 copper layers, 116.8 x 104.1 mm, 22 parts, among them J1 Mouting_Screw_3mm, J2 Mouting_Screw_3mm, J3 Mouting_Screw_3mm

Commit message: Met à jour le PCB kicad DISCO F746 NG
Parts:
- BLE1: value Conn_01x05 -> Conn_01x06; footprint Connector_PinHeader_2.54mm:PinHeader_1x05_P2.54mm_Vertical -> Connector_PinHeader_2.54mm:PinHeader_1x06_P2.54mm_Vertical
- moved BLE1 2.54 mm to (188.0, 137.2)
Connections:
- A2 pad 23: unconnected-(A2-Pad23) -> /STATE_BLE_PI2
- BLE1 pad 1: /5V_BLE/MOT -> unconnected-(BLE1-Pad1)
- BLE1 pad 2: GND -> /5V_BLE/MOT
- BLE1 pad 3: /TX_BLE_PC6 -> GND
- BLE1 pad 4: /RX_BLE_PC7 -> /TX_BLE_PC6
- BLE1 pad 5: unconnected-(BLE1-Pad5) -> /RX_BLE_PC7
Routing:
- net /STATE_BLE_PI2: track 0.00 -> 77.1 mm, vias 0 -> 2
- net GND: track 426.8 -> 370.1 mm, vias 6 -> 4
Other:
- board text added: "ALIM B1-G"
- board text added: "ALIM B2-G"
- board text added: "ALIM B3-G"
- board text added: "G-ALIM A1"
- board text added: "G-ALim A3"
- board text added: "G-BLUETOOTH"
- board text added: "G-LIDAR"
- board text added: "G-PING 1"
- board text added: "G-PING 2"
- board text added: "G-PING 3"
- board text added: "G-PING 4"
- board text added: "G-PING 5"
- board text added: "INFRA 1-V"
- board text added: "INFRA 2-V"
- board text added: "INFRA 3-V"
- board text added: "MOTEUR-G"
- board text added: "SERVO-G"
- board text removed: "ALIM A1"
- board text removed: "ALIM B1"
- board text removed: "ALIM B2"
- board text removed: "ALIM B3"
- board text removed: "ALim A3"
- board text removed: "BLUETOOTH"
- board text removed: "INFRA 1"
- board text removed: "INFRA 2"
- board text removed: "INFRA 3"
- board text removed: "LIDAR"
- board text removed: "MOTEUR"
- board text removed: "PING 1"
- board text removed: "PING 2"
- board text removed: "PING 3"
- board text removed: "PING 4"
- board text removed: "PING 5"
- board text removed: "SERVO"

Commit message: MAJ le PCB
Other:
- board text added: "SaphTeamRacing - Carte adaptation"
Changed lines of the file:
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@@
     (effects (font (size 1.5 1.5) (thickness 0.15)))
+  )
+  (gr_text "SaphTeamRacing - Carte adaptation" (at 142.24 73.66) (layer "Eco1.User")
+    (effects (font (size 2 2) (thickness 0.15)))
   )
   (gr_text "G-PING 3\n" (at 206.243166 114.488254) (layer "Eco1.User")

Commit message: MAJ le PCB
Connections:
- net /I1_PA0 renamed /I1
- net /I2_PF10 renamed /I2
- net /I3_PF9 renamed /I3
- net /M_Cmd_PB8 renamed /M_Cmd
- net /P1_PG6 renamed /P1
- net /P2_PB4 renamed /P2
- net /P3_PG7 renamed /P3
- net /P4_PI0 renamed /P4
- net /P5_PH6 renamed /P5
- net /PWM_Lidar_PF8 renamed /PWM_Lidar
- net /RX_BLE_PC7 renamed /RX_BLE
- net /RX_Lidar_PF6 renamed /RX_Lidar
- net /STATE_BLE_PI2 renamed /STATE_BLE
- net /Servo_Cmd_PB14 renamed /Servo_Cmd
- net /TX_BLE_PC6 renamed /TX_BLE
- net /TX_Lidar_PF7 renamed /TX_Lidar
- net /Trig_Cmd_PI_3 renamed /Trig_Cmd

Commit message: MAJ le PCB
Parts:
- moved BLE1 12.7 mm to (200.7, 137.2), turned to -90 degrees
- moved Moteur1 5.08 mm to (190.5, 144.8), turned to 90 degrees
- turned B2 to -90 degrees
Connections:
- A2 pad 13: /TX_Lidar -> /RX_Lidar
- A2 pad 14: /RX_Lidar -> /TX_Lidar
- A2 pad 15: /RX_BLE -> /TX_BLE
- A2 pad 16: /TX_BLE -> /RX_BLE
Routing:
- net /STATE_BLE: track 77.1 -> 54.3 mm, vias 2 -> 0
- net /M_Cmd: track 82.8 -> 98.3 mm
- net /RX_BLE: track 54.2 -> 39.7 mm
- net GND: track 370.1 -> 380.9 mm
- net /TX_Lidar: track 31.9 -> 28.6 mm
- net /TX_BLE: track 42.6 -> 39.7 mm
- net /RX_Lidar: track 30.4 -> 32.2 mm, vias 2 -> 0
- net /5V_BLE/MOT: track 13.8 -> 14.8 mm
- removed copper zone on B.Cu, net GND
- removed copper zone on F.Cu, net GND
Other:
- board text added: "BLUETOOTH-G"
- board text added: "G-ALIM B2"
- board text added: "G-MOTEUR"
- board text removed: "ALIM B2-G"
- board text removed: "G-BLUETOOTH"
- board text removed: "MOTEUR-G"
