File: PCB_DiscoF746-NG/carte_kicad_F46NG/carte_kicad_F46NG.kicad_sch (KiCad schematic)
At the start: 22 parts, among them J1 Mouting_Screw_3mm, J2 Mouting_Screw_3mm, J3 Mouting_Screw_3mm

Commit message: MAJ le PCB
Connections:
- net I1_PA0 renamed I1
- net I2_PF10 renamed I2
- net I3_PF9 renamed I3
- net M_Cmd_PB8 renamed M_Cmd
- net P1_PG6 renamed P1
- net P2_PB4 renamed P2
- net P3_PG7 renamed P3
- net P4_PI0 renamed P4
- net P5_PH6 renamed P5
- net PWM_Lidar_PF8 renamed PWM_Lidar
- net RX_BLE_PC7 renamed RX_BLE
- net RX_Lidar_PF6 renamed RX_Lidar
- net STATE_BLE_PI2 renamed STATE_BLE
- net Servo_Cmd_PB14 renamed Servo_Cmd
- net TX_BLE_PC6 renamed TX_BLE
- net TX_Lidar_PF7 renamed TX_Lidar
- net Trig_Cmd_PI_3 renamed Trig_Cmd
Changed lines of the file:
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@@
     (effects (font (size 1.27 1.27)) (justify right bottom))
   )
-  (label "P3_PG7" (at 43.18 45.72 0)
+  (label "P3" (at 43.18 45.72 0)
     (effects (font (size 1.27 1.27)) (justify left bottom))
   )
-  (label "Servo_Cmd_PB14" (at 207.01 29.21 180)
+  (label "Servo_Cmd" (at 207.01 29.21 180)
     (effects (font (size 1.27 1.27)) (justify right bottom))
   )
-  (label "Trig_Cmd_PI_3" (at 43.18 40.64 0)
+  (label "Trig_Cmd" (at 43.18 40.64 0)
     (effects (font (size 1.27 1.27)) (justify left bottom))
   )
-  (label "TX_BLE_PC6" (at 165.1 63.5 180)
+  (label "TX_BLE" (at 165.1 63.5 180)
     (effects (font (size 1.27 1.27)) (justify right bottom))
   )
-  (label "P1_PG6" (at 43.18 43.18 0)
+  (label "P1" (at 43.18 43.18 0)
     (effects (font (size 1.27 1.27)) (justify left bottom))
   )
-  (label "I3_PF9" (at 66.04 173.99 180)
+  (label "I3" (at 66.04 173.99 180)
     (effects (font (size 1.27 1.27)) (justify right bottom))
   )
@@
     (effects (font (size 1.27 1.27)) (justify right bottom))
   )
-  (label "P4_PI0" (at 39.37 119.38 0)
+  (label "P4" (at 39.37 119.38 0)
     (effects (font (size 1.27 1.27)) (justify left bottom))
   )
-  (label "RX_Lidar_PF6" (at 152.4 27.94 180)
+  (label "RX_Lidar" (at 152.4 27.94 180)
     (effects (font (size 1.27 1.27)) (justify right bottom))
   )
-  (label "Trig_Cmd_PI_3" (at 76.2 118.11 0)
+  (label "Trig_Cmd" (at 76.2 118.11 0)
     (effects (font (size 1.27 1.27)) (justify left bottom))
   )
-  (label "P2_PB4" (at 43.18 48.26 0)
+  (label "P2" (at 43.18 48.26 0)
     (effects (font (size 1.27 1.27)) (justify left bottom))
   )
-  (label "P5_PH6" (at 39.37 104.14 0)
+  (label "P5" (at 39.37 104.14 0)
     (effects (font (size 1.27 1.27)) (justify left bottom))
   )
-  (label "TX_Lidar_PF7" (at 116.84 60.96 180)
+  (label "TX_Lidar" (at 116.84 60.96 180)
     (effects (font (size 1.27 1.27)) (justify right bottom))
   )
@@
     (effects (font (size 1.27 1.27)) (justify right bottom))
   )
-  (label "PWM_Lidar_PF8" (at 152.4 33.02 180)
+  (label "PWM_Lidar" (at 152.4 33.02 180)
     (effects (font (size 1.27 1.27)) (justify right bottom))
   )
-  (label "I1_PA0" (at 105.41 55.88 180)
+  (label "I1" (at 105.41 55.88 180)
     (effects (font (size 1.27 1.27)) (justify right bottom))
   )
-  (label "P3_PG7" (at 39.37 135.89 0)
+  (label "P3" (at 39.37 135.89 0)
     (effects (font (size 1.27 1.27)) (justify left bottom))
   )
@@
     (effects (font (size 1.27 1.27)) (justify right bottom))
   )
-  (label "STATE_BLE_PI2" (at 43.18 55.88 0)
+  (label "STATE_BLE" (at 43.18 55.88 0)
     (effects (font (size 1.27 1.27)) (justify left bottom))
   )
@@
     (effects (font (size 1.27 1.27)) (justify right bottom))
   )
-  (label "Servo_Cmd_PB14" (at 39.37 66.04 0)
+  (label "Servo_Cmd" (at 39.37 66.04 0)
     (effects (font (size 1.27 1.27)) (justify left bottom))
   )
@@
     (effects (font (size 1.27 1.27)) (justify right bottom))
   )
-  (label "Trig_Cmd_PI_3" (at 35.56 133.35 0)
+  (label "Trig_Cmd" (at 35.56 133.35 0)
     (effects (font (size 1.27 1.27)) (justify left bottom))
   )
-  (label "RX_BLE_PC7" (at 165.1 66.04 180)
+  (label "RX_BLE" (at 165.1 66.04 180)
     (effects (font (size 1.27 1.27)) (justify right bottom))
   )
-  (label "I3_PF9" (at 105.41 50.8 180)
+  (label "I3" (at 105.41 50.8 180)
     (effects (font (size 1.27 1.27)) (justify right bottom))
   )
-  (label "M_Cmd_PB8" (at 207.01 40.64 180)
+  (label "M_Cmd" (at 207.01 40.64 180)
     (effects (font (size 1.27 1.27)) (justify right bottom))
   )
-  (label "Trig_Cmd_PI_3" (at 76.2 101.6 0)
+  (label "Trig_Cmd" (at 76.2 101.6 0)
     (effects (font (size 1.27 1.27)) (justify left bottom))
   )
-  (label "P2_PB4" (at 80.01 104.14 0)
+  (label "P2" (at 80.01 104.14 0)
     (effects (font (size 1.27 1.27)) (justify left bottom))
   )
@@
     (effects (font (size 1.27 1.27)) (justify right bottom))
   )
-  (label "Trig_Cmd_PI_3" (at 35.56 101.6 0)
+  (label "Trig_Cmd" (at 35.56 101.6 0)
     (effects (font (size 1.27 1.27)) (justify left bottom))
   )
-  (label "Trig_Cmd_PI_3" (at 35.56 116.84 0)
+  (label "Trig_Cmd" (at 35.56 116.84 0)
     (effects (font (size 1.27 1.27)) (justify left bottom))
   )
-  (label "P4_PI0" (at 43.18 50.8 0)
+  (label "P4" (at 43.18 50.8 0)
     (effects (font (size 1.27 1.27)) (justify left bottom))
   )
-  (label "TX_Lidar_PF7" (at 152.4 25.4 180)
+  (label "TX_Lidar" (at 152.4 25.4 180)
     (effects (font (size 1.27 1.27)) (justify right bottom))
   )
-  (label "RX_Lidar_PF6" (at 116.84 63.5 180)
+  (label "RX_Lidar" (at 116.84 63.5 180)
     (effects (font (size 1.27 1.27)) (justify right bottom))
   )
-  (label "P5_PH6" (at 43.18 53.34 0)
+  (label "P5" (at 43.18 53.34 0)
     (effects (font (size 1.27 1.27)) (justify left bottom))
   )
@@
     (effects (font (size 1.27 1.27)) (justify right bottom))
   )
-  (label "P1_PG6" (at 80.01 120.65 0)
+  (label "P1" (at 80.01 120.65 0)
     (effects (font (size 1.27 1.27)) (justify left bottom))
   )
-  (label "TX_BLE_PC6" (at 43.18 38.1 0)
+  (label "TX_BLE" (at 43.18 38.1 0)
     (effects (font (size 1.27 1.27)) (justify left bottom))
   )
-  (label "STATE_BLE_PI2" (at 153.67 68.58 0)
+  (label "STATE_BLE" (at 153.67 68.58 0)
     (effects (font (size 1.27 1.27)) (justify left bottom))
   )
@@
     (effects (font (size 1.27 1.27)) (justify right bottom))
   )
-  (label "PWM_Lidar_PF8" (at 116.84 58.42 180)
+  (label "PWM_Lidar" (at 116.84 58.42 180)
     (effects (font (size 1.27 1.27)) (justify right bottom))
   )
@@
     (effects (font (size 1.27 1.27)) (justify right bottom))
   )
-  (label "I1_PA0" (at 66.04 151.13 180)
+  (label "I1" (at 66.04 151.13 180)
     (effects (font (size 1.27 1.27)) (justify right bottom))
   )
-  (label "I2_PF10" (at 105.41 53.34 180)
+  (label "I2" (at 105.41 53.34 180)
     (effects (font (size 1.27 1.27)) (justify right bottom))
   )
@@
     (effects (font (size 1.27 1.27)) (justify right bottom))
   )
-  (label "RX_BLE_PC7" (at 43.18 35.56 0)
+  (label "RX_BLE" (at 43.18 35.56 0)
     (effects (font (size 1.27 1.27)) (justify left bottom))
   )
@@
     (effects (font (size 1.27 1.27)) (justify right bottom))
   )
-  (label "I2_PF10" (at 66.04 162.56 180)
+  (label "I2" (at 66.04 162.56 180)
     (effects (font (size 1.27 1.27)) (justify right bottom))
   )
-  (label "M_Cmd_PB8" (at 115.57 71.12 180)
+  (label "M_Cmd" (at 115.57 71.12 180)
     (effects (font (size 1.27 1.27)) (justify right bottom))
   )

Commit message: MAJ le PCB
Parts:
- renumbered BLE to BLE1
Changed lines of the file:
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@@
   (symbol (lib_id "power:GND") (at 148.59 60.96 270) (unit 1)
     (in_bom yes) (on_board yes) (fields_autoplaced)
-    (property "Reference" "#PWR?" (id 0) (at 142.24 60.96 0)
+    (property "Reference" "#PWR0102" (id 0) (at 142.24 60.96 0)
       (effects (font (size 1.27 1.27)) hide)
     )
@@
   (symbol (lib_id "Connector_Generic:Conn_01x06") (at 182.88 60.96 0) (unit 1)
     (in_bom yes) (on_board yes) (fields_autoplaced)
-    (property "Reference" "BLE" (id 0) (at 185.42 60.9599 0)
+    (property "Reference" "BLE1" (id 0) (at 185.42 60.9599 0)
       (effects (font (size 1.27 1.27)) (justify left))
     )
@@
       (reference "#PWR0101") (unit 1) (value "GND") (footprint "")
     )
+    (path "/6e413ce5-ddaf-479d-ab31-d32d62b0c2f3"
+      (reference "#PWR0102") (unit 1) (value "GND") (footprint "")
+    )
     (path "/ac288dec-f1d0-42f2-a16f-dee351c36ca1"
       (reference "#PWR0103") (unit 1) (value "GND") (footprint "")
@@
       (reference "#PWR0119") (unit 1) (value "GND") (footprint "")
     )
-    (path "/6e413ce5-ddaf-479d-ab31-d32d62b0c2f3"
-      (reference "#PWR?") (unit 1) (value "GND") (footprint "")
-    )
     (path "/f87ce03a-03d7-4533-9c1c-b0f2552e1cd0"
       (reference "A1") (unit 1) (value "Conn_01x02") (footprint "Connector_PinHeader_2.54mm:PinHeader_1x02_P2.54mm_Vertical")
@@
     )
     (path "/7b98ef29-43ae-47e9-9801-dab1ae51395e"
-      (reference "BLE") (unit 1) (value "Conn_01x06") (footprint "Connector_PinHeader_2.54mm:PinHeader_1x06_P2.54mm_Vertical")
+      (reference "BLE1") (unit 1) (value "Conn_01x06") (footprint "Connector_PinHeader_2.54mm:PinHeader_1x06_P2.54mm_Vertical")
     )
     (path "/6c9a076d-21ce-48cc-a4d7-55822e95fa95"

Commit message: MAJ le PCB
Connections:
- net RX_BLE: now also A2.16 (D1/TX); no longer A2.15 (D0/RX)
- net RX_Lidar: now also A2.13 (SDA/A4); no longer A2.14 (SCL/A5)
- net TX_BLE: now also A2.15 (D0/RX); no longer A2.16 (D1/TX)
- net TX_Lidar: now also A2.14 (SCL/A5); no longer A2.13 (SDA/A4)
Changed lines of the file:
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@@
   (junction (at 73.66 78.74) (diameter 0) (color 0 0 0 0)
   )
+  (wire (pts (xy 83.82 63.5) (xy 116.84 63.5))
+    (stroke (width 0) (type default) (color 0 0 0 0))
+  )
   (wire (pts (xy 83.82 55.88) (xy 105.41 55.88))
     (stroke (width 0) (type default) (color 0 0 0 0))
@@
     (stroke (width 0) (type default) (color 0 0 0 0))
   )
+  (wire (pts (xy 43.18 35.56) (xy 58.42 35.56))
+    (stroke (width 0) (type default) (color 0 0 0 0))
+  )
   (wire (pts (xy 35.56 133.35) (xy 50.8 133.35))
     (stroke (width 0) (type default) (color 0 0 0 0))
@@
     (stroke (width 0) (type default) (color 0 0 0 0))
   )
+  (wire (pts (xy 43.18 50.8) (xy 58.42 50.8))
+    (stroke (width 0) (type default) (color 0 0 0 0))
+  )
+  (wire (pts (xy 39.37 135.89) (xy 50.8 135.89))
+    (stroke (width 0) (type default) (color 0 0 0 0))
+  )
+  (wire (pts (xy 158.75 30.48) (xy 134.62 30.48))
+    (stroke (width 0) (type default) (color 0 0 0 0))
+  )
+  (wire (pts (xy 207.01 38.1) (xy 209.55 38.1))
+    (stroke (width 0) (type default) (color 0 0 0 0))
+  )
+  (wire (pts (xy 204.47 105.41) (xy 209.55 105.41))
+    (stroke (width 0) (type default) (color 0 0 0 0))
+  )
+  (wire (pts (xy 243.84 83.82) (xy 248.92 83.82))
+    (stroke (width 0) (type default) (color 0 0 0 0))
+  )
+  (wire (pts (xy 45.72 114.3) (xy 50.8 114.3))
+    (stroke (width 0) (type default) (color 0 0 0 0))
+  )
+  (wire (pts (xy 83.82 53.34) (xy 105.41 53.34))
+    (stroke (width 0) (type default) (color 0 0 0 0))
+  )
+  (wire (pts (xy 45.72 130.81) (xy 50.8 130.81))
+    (stroke (width 0) (type default) (color 0 0 0 0))
+  )
+  (wire (pts (xy 142.24 90.17) (xy 142.24 97.79))
+    (stroke (width 0) (type default) (color 0 0 0 0))
+  )
+  (wire (pts (xy 191.77 35.56) (xy 209.55 35.56))
+    (stroke (width 0) (type default) (color 0 0 0 0))
+  )
+  (wire (pts (xy 76.2 118.11) (xy 91.44 118.11))
+    (stroke (width 0) (type default) (color 0 0 0 0))
+  )
+  (wire (pts (xy 165.1 63.5) (xy 177.8 63.5))
+    (stroke (width 0) (type default) (color 0 0 0 0))
+  )
+  (wire (pts (xy 152.4 25.4) (xy 158.75 25.4))
+    (stroke (width 0) (type default) (color 0 0 0 0))
+  )
+  (wire (pts (xy 252.73 111.76) (xy 262.89 111.76))
+    (stroke (width 0) (type default) (color 0 0 0 0))
+  )
+  (wire (pts (xy 72.39 165.1) (xy 55.88 165.1))
+    (stroke (width 0) (type default) (color 0 0 0 0))
+  )
+  (wire (pts (xy 87.63 123.19) (xy 87.63 124.46))
+    (stroke (width 0) (type default) (color 0 0 0 0))
+  )
+  (wire (pts (xy 72.39 153.67) (xy 55.88 153.67))
+    (stroke (width 0) (type default) (color 0 0 0 0))
+  )
+  (wire (pts (xy 152.4 27.94) (xy 158.75 27.94))
+    (stroke (width 0) (type default) (color 0 0 0 0))
+  )
+  (wire (pts (xy 83.82 60.96) (xy 116.84 60.96))
+    (stroke (width 0) (type default) (color 0 0 0 0))
+  )
+  (wire (pts (xy 66.04 167.64) (xy 72.39 167.64))
+    (stroke (width 0) (type default) (color 0 0 0 0))
+  )
+  (wire (pts (xy 168.91 58.42) (xy 177.8 58.42))
+    (stroke (width 0) (type default) (color 0 0 0 0))
+  )
+  (wire (pts (xy 142.24 97.79) (xy 142.24 105.41))
+    (stroke (width 0) (type default) (color 0 0 0 0))
+  )
+  (wire (pts (xy 66.04 173.99) (xy 72.39 173.99))
+    (stroke (width 0) (type default) (color 0 0 0 0))
+  )
+  (wire (pts (xy 66.04 156.21) (xy 72.39 156.21))
+    (stroke (width 0) (type default) (color 0 0 0 0))
+  )
   (wire (pts (xy 43.18 38.1) (xy 58.42 38.1))
     (stroke (width 0) (type default) (color 0 0 0 0))
   )
-  (wire (pts (xy 43.18 50.8) (xy 58.42 50.8))
-    (stroke (width 0) (type default) (color 0 0 0 0))
-  )
-  (wire (pts (xy 39.37 135.89) (xy 50.8 135.89))
-    (stroke (width 0) (type default) (color 0 0 0 0))
-  )
-  (wire (pts (xy 158.75 30.48) (xy 134.62 30.48))
-    (stroke (width 0) (type default) (color 0 0 0 0))
-  )
-  (wire (pts (xy 207.01 38.1) (xy 209.55 38.1))
-    (stroke (width 0) (type default) (color 0 0 0 0))
-  )
-  (wire (pts (xy 204.47 105.41) (xy 209.55 105.41))
-    (stroke (width 0) (type default) (color 0 0 0 0))
-  )
-  (wire (pts (xy 243.84 83.82) (xy 248.92 83.82))
-    (stroke (width 0) (type default) (color 0 0 0 0))
-  )
-  (wire (pts (xy 45.72 114.3) (xy 50.8 114.3))
-    (stroke (width 0) (type default) (color 0 0 0 0))
-  )
-  (wire (pts (xy 83.82 53.34) (xy 105.41 53.34))
-    (stroke (width 0) (type default) (color 0 0 0 0))
-  )
-  (wire (pts (xy 45.72 130.81) (xy 50.8 130.81))
-    (stroke (width 0) (type default) (color 0 0 0 0))
-  )
-  (wire (pts (xy 142.24 90.17) (xy 142.24 97.79))
-    (stroke (width 0) (type default) (color 0 0 0 0))
-  )
-  (wire (pts (xy 191.77 35.56) (xy 209.55 35.56))
-    (stroke (width 0) (type default) (color 0 0 0 0))
-  )
-  (wire (pts (xy 76.2 118.11) (xy 91.44 118.11))
-    (stroke (width 0) (type default) (color 0 0 0 0))
-  )
-  (wire (pts (xy 165.1 63.5) (xy 177.8 63.5))
-    (stroke (width 0) (type default) (color 0 0 0 0))
-  )
-  (wire (pts (xy 152.4 25.4) (xy 158.75 25.4))
-    (stroke (width 0) (type default) (color 0 0 0 0))
-  )
-  (wire (pts (xy 252.73 111.76) (xy 262.89 111.76))
-    (stroke (width 0) (type default) (color 0 0 0 0))
-  )
-  (wire (pts (xy 72.39 165.1) (xy 55.88 165.1))
-    (stroke (width 0) (type default) (color 0 0 0 0))
-  )
-  (wire (pts (xy 87.63 123.19) (xy 87.63 124.46))
-    (stroke (width 0) (type default) (color 0 0 0 0))
-  )
-  (wire (pts (xy 72.39 153.67) (xy 55.88 153.67))
-    (stroke (width 0) (type default) (color 0 0 0 0))
-  )
-  (wire (pts (xy 152.4 27.94) (xy 158.75 27.94))
-    (stroke (width 0) (type default) (color 0 0 0 0))
-  )
-  (wire (pts (xy 43.18 35.56) (xy 58.42 35.56))
-    (stroke (width 0) (type default) (color 0 0 0 0))
-  )
-  (wire (pts (xy 66.04 167.64) (xy 72.39 167.64))
-    (stroke (width 0) (type default) (color 0 0 0 0))
-  )
-  (wire (pts (xy 168.91 58.42) (xy 177.8 58.42))
-    (stroke (width 0) (type default) (color 0 0 0 0))
-  )
-  (wire (pts (xy 142.24 97.79) (xy 142.24 105.41))
-    (stroke (width 0) (type default) (color 0 0 0 0))
-  )
-  (wire (pts (xy 66.04 173.99) (xy 72.39 173.99))
-    (stroke (width 0) (type default) (color 0 0 0 0))
-  )
-  (wire (pts (xy 66.04 156.21) (xy 72.39 156.21))
-    (stroke (width 0) (type default) (color 0 0 0 0))
-  )
   (wire (pts (xy 152.4 33.02) (xy 158.75 33.02))
     (stroke (width 0) (type default) (color 0 0 0 0))
@@
     (stroke (width 0) (type default) (color 0 0 0 0))
   )
-  (wire (pts (xy 83.82 63.5) (xy 116.84 63.5))
-    (stroke (width 0) (type default) (color 0 0 0 0))
-  )
   (wire (pts (xy 43.18 53.34) (xy 58.42 53.34))
     (stroke (width 0) (type default) (color 0 0 0 0))
@@
     (stroke (width 0) (type default) (color 0 0 0 0))
   )
-  (wire (pts (xy 83.82 60.96) (xy 116.84 60.96))
-    (stroke (width 0) (type default) (color 0 0 0 0))
-  )
   (wire (pts (xy 39.37 119.38) (xy 50.8 119.38))
     (stroke (width 0) (type default) (color 0 0 0 0))
@@
     (effects (font (size 1.27 1.27)) (justify left bottom))
   )
-  (label "TX_Lidar" (at 116.84 60.96 180)
+  (label "TX_Lidar" (at 116.84 63.5 180)
     (effects (font (size 1.27 1.27)) (justify right bottom))
   )
@@
     (effects (font (size 1.27 1.27)) (justify right bottom))
   )
-  (label "RX_Lidar" (at 116.84 63.5 180)
+  (label "RX_Lidar" (at 116.84 60.96 180)
     (effects (font (size 1.27 1.27)) (justify right bottom))
   )
@@
     (effects (font (size 1.27 1.27)) (justify left bottom))
   )
-  (label "TX_BLE" (at 43.18 38.1 0)
+  (label "TX_BLE" (at 43.18 35.56 0)
     (effects (font (size 1.27 1.27)) (justify left bottom))
   )
@@
     (effects (font (size 1.27 1.27)) (justify right bottom))
   )
-  (label "RX_BLE" (at 43.18 35.56 0)
-    (effects (font (size 1.27 1.27)) (justify left bottom))
-  )
+  (label "RX_BLE" (at 43.18 38.1 0)
+    (effects (font (size 1.27 1.27)) (justify left bottom))
+  )
